Commit message: fix(simulator): 重构机器人模型坐标系统 — 删除 base_origin，base_link 作为根
移除 URDF 转换遗留的 base_origin/base_link 分离结构。base_link 现在是
承载车身几何、惯量和所有 joint 的根 link，Gazebo 的 OdometryPublisher
直接上报 base_link 位姿，消除了原本需要在 C++ 层补偿的 0.75m z 偏移。

## 模型改动 (model.sdf.xacro)

**结构变更：**
- 删除 base_origin link（原实体根 link）
- 删除 base_origin_to_base_link fixed joint
- 删除旧 base_link（质量 0.001kg 的空壳）
- 新 base_link 继承原 base_origin 的全部几何、惯量、传感器

**坐标调整（新原点下移 0.75m，所有 z +0.75）：**
- 车身惯量 pose：-0.56 → 0.19
- 车身碰撞/视觉 pose：-0.5 → 0.25
- 轮子轴心：-0.6 → 0.15（即 ${wheel_radius}，自解释）
- LiDAR mount property：-0.27 → 0.48
- LiDAR support visual 计算公式：-0.5 → 0.25（车身几何中心）

**parent 修改：**
- 四个轮子 joint parent：base_origin → base_link
- LiDAR joint parent：base_origin → base_link

**注释更新：**
- 轮子宏注释反映新语义（base_link 在地面，轴心在轮半径高度）

## Launch 文件改动

**robot.launch.py & pointcloud_complete_launch.py：**
- 函数调用：generate_robot_sdf_from_xmacro → generate_robot_sdf
- 文件路径：model.sdf.xmacro → model.sdf.xacro

## 出生位姿调整 (world 文件)

模型原点下移 0.75m，spawn pose 相应调整（z -0.75）：
- flat_small_scale_maze：z 0.75 → 0.0
- map_desert：z 2.509 → 1.759
- map_hill：z 0.750 → 0.0
- map_vocano：z 3.917 → 3.167

## URDF 修复 (sdf_launch_utils.py)

**normalize_robot_urdf_for_rviz() 重新实现：**
- 修复 SDF→URDF 转换问题：轮子 pose 错误地放在 <link><origin>
- 将 link origin 的 xyz 移到 joint origin（URDF 标准位置）
- 将 link origin 的 rpy 移到 visual/collision origin（保持几何朝向）
- 确保 RViz2 正确显示轮子位置和方向

## 验证结果

- ✓ Xacro 展开：8 links（减 1），7 joints（减 2）
- ✓ base_link 包含 collision、visual、inertial
- ✓ 所有轮子 joint parent 正确指向 base_link
- ✓ 编译通过
- ✓ Gazebo spawn：机器人贴地，无浮空，无掉落
- ✓ /odom position.z ≈ 0（平地上，误差 ±0.001）
- ✓ RViz2 RobotModel 显示正常，轮子位置和方向正确
- ✓ TF 树无 base_origin frame

File: finenav_simulator/resource/robot/model.sdf.xacro (robot description, xacro)
@@ -16,5 +16,5 @@
     <xacro:property name="lidar_mount_x" value="0.16"/>
     <xacro:property name="lidar_mount_y" value="0.0"/>
-    <xacro:property name="lidar_mount_z" value="-0.27"/>
+    <xacro:property name="lidar_mount_z" value="0.48"/>
     <xacro:property name="lidar_mount_pitch" value="0.78539816339"/>
     <xacro:property name="lidar_mount_slide_along_slope" value="0.045"/>
@@ -60,8 +60,6 @@
          wheel's geometry, mass or contact parameters once and all four follow.
          `flip` is +1 on the left and -1 on the right, mirroring the cylinder
-         about the x axis.  The wheel links parent to `base_origin` because that
-         is where the chassis inertia lives; keep it that way or the physics
-         changes.  z = -0.6 is base_origin -> base_link (-0.75) plus the wheel
-         radius, i.e. axles sit one radius above base_link. -->
+         about the x axis.  The wheel links parent to `base_link`, which sits at
+         ground level, so axles are positioned at exactly ${wheel_radius}. -->
     <xacro:macro name="wheel" params="name x y flip">
         <frame name="${name}_frame" attached_to="base_link">
@@ -70,5 +68,5 @@
         <frame name="${name}_wheel" attached_to="${name}_frame"/>
         <link name="${name}_link">
-            <pose relative_to="base_origin">${x} ${y} -0.6 ${flip * 1.57} 0 0</pose>
+            <pose relative_to="base_link">${x} ${y} ${wheel_radius} ${flip * 1.57} 0 0</pose>
             <inertial>
                 <mass>0.75</mass>
@@ -125,5 +123,5 @@
         </link>
         <joint name="${name}_joint" type="revolute">
-            <parent>base_origin</parent>
+            <parent>base_link</parent>
             <child>${name}_link</child>
             <axis>
@@ -143,7 +141,7 @@
     </xacro:macro>
     <model name="robot">
-        <link name="base_origin">
-            <inertial>
-                <pose>0 0 -0.56 0 0 0</pose>
+        <link name="base_link">
+            <inertial>
+                <pose>0 0 0.19 0 0 0</pose>
                 <mass>${base_mass}</mass>
                 <inertia>
@@ -157,5 +155,5 @@
             </inertial>
             <collision name="base_collision">
-                <pose>0 0 -0.5 0 0 0</pose>
+                <pose>0 0 0.25 0 0 0</pose>
                 <geometry>
                     <box>
@@ -164,6 +162,6 @@
                 </geometry>
             </collision>
-            <visual name="base_origin_fixed_joint_lump__base_link_visual_1">
-                <pose>0 0 -0.5 0 0 0</pose>
+            <visual name="base_visual">
+                <pose>0 0 0.25 0 0 0</pose>
                 <geometry>
                     <box>
@@ -186,5 +184,5 @@
         </link>
         <link name="base_lidar">
-            <pose relative_to="base_origin">${lidar_mount_x + lidar_mount_slide_along_slope * cos(lidar_mount_pitch)} ${lidar_mount_y} ${lidar_mount_z - lidar_mount_slide_along_slope * sin(lidar_mount_pitch)} 0 ${lidar_mount_pitch} 0</pose>
+            <pose relative_to="base_link">${lidar_mount_x + lidar_mount_slide_along_slope * cos(lidar_mount_pitch)} ${lidar_mount_y} ${lidar_mount_z - lidar_mount_slide_along_slope * sin(lidar_mount_pitch)} 0 ${lidar_mount_pitch} 0</pose>
             <inertial>
                 <pose>0 0 ${lidar_visual_z} 0 0 0</pose>
@@ -214,5 +212,5 @@
             </visual>
             <visual name="base_lidar_support_visual">
-                <pose>${((lidar_visual_z - lidar_length / 2.0 - lidar_support_lidar_clearance - lidar_support_height / sqrt(2.0) - lidar_support_body_clearance) - (((-0.5 + base_height / 2.0) - (lidar_mount_z - lidar_mount_slide_along_slope * sin(lidar_mount_pitch))) / cos(lidar_mount_pitch))) / tan(lidar_mount_pitch) + lidar_support_x_offset} ${lidar_support_y} ${lidar_visual_z - lidar_length / 2.0 - lidar_support_lidar_clearance + lidar_support_z_offset} 0 ${lidar_support_pitch} 0</pose>
+                <pose>${((lidar_visual_z - lidar_length / 2.0 - lidar_support_lidar_clearance - lidar_support_height / sqrt(2.0) - lidar_support_body_clearance) - (((0.25 + base_height / 2.0) - (lidar_mount_z - lidar_mount_slide_along_slope * sin(lidar_mount_pitch))) / cos(lidar_mount_pitch))) / tan(lidar_mount_pitch) + lidar_support_x_offset} ${lidar_support_y} ${lidar_visual_z - lidar_length / 2.0 - lidar_support_lidar_clearance + lidar_support_z_offset} 0 ${lidar_support_pitch} 0</pose>
                 <geometry>
                     <mesh>
@@ -270,25 +268,7 @@
         </link>
         <joint name="base_lidar_joint" type="fixed">
-            <parent>base_origin</parent>
+            <parent>base_link</parent>
             <child>base_lidar</child>
             <pose>${lidar_mount_x + lidar_mount_slide_along_slope * cos(lidar_mount_pitch)} ${lidar_mount_y} ${lidar_mount_z - lidar_mount_slide_along_slope * sin(lidar_mount_pitch)} 0 ${lidar_mount_pitch} 0</pose>
-        </joint>
-        <link name="base_link">
-            <inertial>
-                <mass>0.001</mass>
-                <inertia>
-                    <ixx>0.000001</ixx>
-                    <iyy>0.000001</iyy>
-                    <izz>0.000001</izz>
-                    <ixy>0</ixy>
-                    <ixz>0</ixz>
-                    <iyz>0</iyz>
-                </inertia>
-            </inertial>
-        </link>
-        <joint name="base_origin_to_base_link" type="fixed">
-            <parent>base_origin</parent>
-            <child>base_link</child>
-            <pose>0 0 -0.75 0 0 0</pose>
         </joint>
         <link name="imu">
